Commit message: correct arm base pose

File: libs/robot_description/rl/bimanual_panda_tesollo_jar.urdf (robot description, URDF)
Before this commit: robot bimanual_panda_tesollo_jar, 62 links, 61 joints
Joints:
- joint left_panda_mount: origin xyz=-0.558 -0.092 0.0 rpy=0 0 0 -> xyz=-0.558 0.092 0.0 rpy=0 0 0
- joint right_panda_mount: origin xyz=0.5588 -0.092 0.0 rpy=0 0 3.14159265359 -> xyz=0.5588 0.092 0.0 rpy=0 0 3.14159265359
