Commit message: transfer table_top to urdf, fix collision detection

File: libs/robot_description/rl/bimanual_panda_tesollo.urdf (robot description, URDF)
Before this commit: robot bimanual_panda_tesollo, 59 links, 58 joints
Links:
- added link table_top; collision box size=1.8288 0.62865 0.045; visual box size=1.8288 0.62865 0.045
Joints:
- added joint table_top_joint: type fixed, parent world, child table_top, origin xyz=0 0 -0.022500 rpy=0 0 0
- joint left_panda_mount: origin xyz=-0.558 -0.092 0.0225 rpy=0 0 0 -> xyz=-0.558 -0.092 0.0 rpy=0 0 0
- joint right_panda_mount: origin xyz=0.5588 -0.092 0.0225 rpy=0 0 3.14159265359 -> xyz=0.5588 -0.092 0.0 rpy=0 0 3.14159265359

Commit message: replay

File: libs/robot_description/rl/bimanual_panda_tesollo.urdf (robot description, URDF)
Before this commit: robot bimanual_panda_tesollo, 60 links, 59 joints
Joints:
- joint left_TIPTOP1: origin xyz=0.058 0 0.002 rpy=0 0 0 -> xyz=0.058 0.005 0.00 rpy=0 0 0
- joint left_TIPTOP2: origin xyz=0.058 0 0.002 rpy=0 0 0 -> xyz=0.058 0.005 0.00 rpy=0 0 0
- joint left_TIPTOP3: origin xyz=0.058 0 0.002 rpy=0 0 0 -> xyz=0.058 0.005 0.00 rpy=0 0 0
- joint left_delto_offset_joint: origin xyz=0 0 0.05 rpy=0 0 0 -> xyz=0 0 0.02 rpy=0 0 0
- joint left_panda_mount: origin xyz=-0.558 -0.092 0.0 rpy=0 0 0 -> xyz=-0.5588 0.092 0.9369 rpy=0 0 0
- joint right_TIPTOP1: origin xyz=0.058 0 0.002 rpy=0 0 0 -> xyz=0.058 0.005 0.00 rpy=0 0 0
- joint right_TIPTOP2: origin xyz=0.058 0 0.002 rpy=0 0 0 -> xyz=0.058 0.005 0.00 rpy=0 0 0
- joint right_TIPTOP3: origin xyz=0.058 0 0.002 rpy=0 0 0 -> xyz=0.058 0.005 0.00 rpy=0 0 0
- joint right_delto_offset_joint: origin xyz=0 0 0.05 rpy=0 0 0 -> xyz=0 0 0.02 rpy=0 0 0
- joint right_panda_mount: origin xyz=0.5588 -0.092 0.0 rpy=0 0 3.14159265359 -> xyz=0.5588 0.092 0.9369 rpy=0 0 3.14159265359
- joint table_top_joint: origin xyz=0 0 -0.022500 rpy=0 0 0 -> xyz=0 0 0.914400 rpy=0 0 0

File: libs/robot_description/rl/panda_w_tesollo.urdf (robot description, URDF)
Before this commit: robot panda_w_tesollo, 29 links, 28 joints
Joints:
- joint TIPTOP1: origin xyz=0.058 0 0.002 rpy=0 0 0 -> xyz=0.058 0.005 0.00 rpy=0 0 0
- joint TIPTOP2: origin xyz=0.058 0 0.002 rpy=0 0 0 -> xyz=0.058 0.005 0.00 rpy=0 0 0
- joint TIPTOP3: origin xyz=0.058 0 0.002 rpy=0 0 0 -> xyz=0.058 0.005 0.00 rpy=0 0 0
- joint delto_offset_joint: origin xyz=0 0 0.05 rpy=0 0 0 -> xyz=0 0 0.02 rpy=0 0 0

Commit message: new urdf to fix flange error

File: libs/robot_description/rl/bimanual_panda_tesollo.urdf (robot description, URDF)
Before this commit: robot bimanual_panda_tesollo, 60 links, 59 joints
Joints:
- joint left_panda_gripper_joint: origin xyz=0 0 0.106 rpy=0 0 -0.785 -> xyz=0 0 0.106 rpy=0 0 -1.015
- joint right_panda_gripper_joint: origin xyz=0 0 0.106 rpy=0 0 -0.785 -> xyz=0 0 0.106 rpy=0 0 -1.015

File: libs/robot_description/rl/panda_w_tesollo.urdf (robot description, URDF)
Before this commit: robot panda_w_tesollo, 29 links, 28 joints
Joints:
- joint panda_gripper_joint: origin xyz=0 0 0.106 rpy=0 0 -0.785 -> xyz=0 0 0.106 rpy=0 0 -1.015
